Commit message: changed slam from slam tool box to cartographer and added rst documentation

File: usv_description/urdf/usv.urdf (robot description, URDF)
Before this commit: robot mbzirc_usv_base, 5 links, 4 joints
Links:
- removed link mbzirc_usv_base__base_link
- removed link mbzirc_usv_base__left_engine_link
- removed link mbzirc_usv_base__left_propeller_link
- removed link mbzirc_usv_base__right_engine_link
- removed link mbzirc_usv_base__right_propeller_link
- added link usv/base_link, mass 727.247; collision box size=0.112524 0.379202 0.0459061; collision box size=0.112524 0.379202 0.0459061
- added link usv/left_engine_link, mass 15.0; visual mesh filename=package://two_wheeled_robot/meshes/motor.dae scale=0.01 0.01 0.01
- added link usv/left_propeller_link, mass 0.5; visual mesh filename=package://two_wheeled_robot/meshes/propeller.dae scale=0.01 0.01 0.01
- added link usv/right_engine_link, mass 15.0; visual mesh filename=package://two_wheeled_robot/meshes/motor.dae scale=0.01 0.01 0.01
- added link usv/right_propeller_link, mass 0.5; visual mesh filename=package://two_wheeled_robot/meshes/propeller.dae scale=0.01 0.01 0.01
Joints:
- removed joint mbzirc_usv_base__left_chassis_engine_joint
- removed joint mbzirc_usv_base__left_engine_propeller_joint
- removed joint mbzirc_usv_base__right_chassis_engine_joint
- removed joint mbzirc_usv_base__right_engine_propeller_joint
- added joint usv/left_chassis_engine_joint: type revolute, parent usv/base_link, child usv/left_engine_link, origin xyz=0     1.348 -0.546 rpy=0      0      1.57079, axis 0 0 1, limit lower=-1.57079 upper=1.57079 effort=10.0 velocity=10.0
- added joint usv/left_engine_propeller_joint: type continuous, parent usv/left_engine_link, child usv/left_propeller_link, origin xyz=0     0.151 -0.17 rpy=0 0 0, axis 0 -1  0, limit lower=0.0 upper=0.0 effort=100.0 velocity=100.0
- added joint usv/right_chassis_engine_joint: type revolute, parent usv/base_link, child usv/right_engine_link, origin xyz=0    -1.348 -0.546 rpy=0      0      1.57079, axis 0 0 1, limit lower=-1.57079 upper=1.57079 effort=10.0 velocity=10.0
- added joint usv/right_engine_propeller_joint: type continuous, parent usv/right_engine_link, child usv/right_propeller_link, origin xyz=0     0.151 -0.17 rpy=0 0 0, axis 0 -1  0, limit lower=0.0 upper=0.0 effort=100.0 velocity=100.0

Commit message: added odometry and custom tf broadcaster for map building

File: usv_description/urdf/usv.urdf (robot description, URDF)
Before this commit: robot usv, 5 links, 4 joints
Links:
- removed link usv/base_link
- removed link usv/left_engine_link
- removed link usv/left_propeller_link
- removed link usv/right_engine_link
- removed link usv/right_propeller_link
- added link usv, mass 727.247; collision box size=0.112524 0.379202 0.0459061; collision box size=0.112524 0.379202 0.0459061
Joints:
- removed joint usv/left_chassis_engine_joint
- removed joint usv/left_engine_propeller_joint
- removed joint usv/right_chassis_engine_joint
- removed joint usv/right_engine_propeller_joint

Commit message: working pid

File: usv_description/urdf/usv.urdf (robot description, URDF)
Before this commit: robot usv_robot, 1 links, 0 joints
Links:
- link usv: geometry collision box size=0.112524 0.379202 0.0459061; collision box size=0.112524 0.379202 0.0459061
